Commit message: Create drivable robot

File: project_4_differential_drive_robot/src/project_4_differential_drive_robot/urdf/components.xacro (robot description, xacro)
@@ -70,4 +70,5 @@
             <axis xyz="0 1 0"/>
             <origin xyz="0 ${reflect * ((wheel_base_width/2) + (wheel_length/2))} 0" rpy="0 0 0"/>
+            <limit velocity="${wheel_max_velocity}" effort="${wheel_max_effort}"/>
         </joint>
     </xacro:macro>

File: project_4_differential_drive_robot/src/project_4_differential_drive_robot/urdf/properties.xacro (robot description, xacro)
@@ -26,3 +26,6 @@
     <!-- Height of base_link origin above the ground -->
     <xacro:property name="base_link_ground_height" value="${(base_height/2) + (wheel_base_height/2) + wheel_radius}"/>
+    <!-- Wheel actuator limits -->
+    <xacro:property name="wheel_max_velocity" value="10.0"/>      <!-- rad/s -->
+    <xacro:property name="wheel_max_effort" value="1.0"/>        <!-- N*m -->
 </robot>
