Commit message: Update physical properties

File: project_6_2r_robot_arm/src/project_6_2r_robot_arm/urdf/2r_robot_arm.urdf.xacro (robot description, xacro)
@@ -3,8 +3,8 @@
   <xacro:include filename="properties.xacro"/>
   <xacro:include filename="components.xacro"/>
-  <!-- Base Footprint -->
-  <link name="base_footprint"/>
-  <joint name="base_footprint_joint" type="fixed">
-    <parent link="base_footprint"/>
+  <!--Attach base_link to world -->
+  <link name="world"/>
+  <joint name="joint_world_base" type="fixed">
+    <parent link="world"/>
     <child link="base_link"/>
     <origin xyz="0 0 0" rpy="0 0 0"/>
@@ -14,24 +14,32 @@
     <visual>
       <origin xyz="0 0 ${base_height / 2.0}"/>
-      <geometry><box size="${base_width} ${base_length} ${base_height}"/></geometry>
+      <geometry>
+        <box size="${base_width} ${base_length} ${base_height}"/>
+      </geometry>
       <material name="base_gray"/>
     </visual>
     <collision>
       <origin xyz="0 0 ${base_height / 2.0}"/>
-      <geometry><box size="${base_width} ${base_length} ${base_height}"/></geometry>
+      <geometry>
+        <box size="${base_width} ${base_length} ${base_height}"/>
+      </geometry>
     </collision>
-    <xacro:box_inertia mass="${base_mass}" x="${base_width}" y="${base_length}" z="${base_height}"/>
+    <xacro:box_inertia origin_xyz="0 0 ${base_height / 2.0}" mass="${base_mass}" base_width="${base_width}" base_length="${base_length}" base_height="${base_height}"/>
   </link>
   <link name="pedestal_link">
     <visual>
       <origin xyz="0 0 ${base_height + pedestal_height / 2.0}"/>
-      <geometry><cylinder length="${pedestal_height}" radius="${pedestal_radius}"/></geometry>
+      <geometry>
+        <cylinder length="${pedestal_height}" radius="${pedestal_radius}"/>
+      </geometry>
       <material name="base_gray"/>
     </visual>
     <collision>
       <origin xyz="0 0 ${base_height + pedestal_height / 2.0}"/>
-      <geometry><cylinder length="${pedestal_height}" radius="${pedestal_radius}"/></geometry>
+      <geometry>
+        <cylinder length="${pedestal_height}" radius="${pedestal_radius}"/>
+      </geometry>
     </collision>
-    <xacro:cylinder_inertia mass="${pedestal_mass}" radius="${pedestal_radius}" length="${pedestal_height}"/>
+    <xacro:z_aligned_cylinder_inertia origin_xyz="0 0 ${base_height + pedestal_height / 2.0}" mass="${pedestal_mass}" radius="${pedestal_radius}" length="${pedestal_height}"/>
   </link>
   <joint name="joint_base_pedestal" type="fixed">
@@ -44,7 +52,16 @@
     <visual>
       <origin xyz="0 0 0" rpy="${pi / 2.0} 0 0"/>
-      <geometry><cylinder radius="${shoulder_radius}" length="${shoulder_length}"/></geometry>
+      <geometry>
+        <cylinder radius="${shoulder_radius}" length="${shoulder_length}"/>
+      </geometry>
       <material name="joint_dark"/>
     </visual>
+    <collision>
+      <origin xyz="0 0 0" rpy="${pi / 2.0} 0 0"/>
+      <geometry>
+        <cylinder radius="${shoulder_radius}" length="${shoulder_length}"/>
+      </geometry>
+    </collision>
+    <xacro:y_aligned_cylinder_inertia origin_xyz="0 0 0" mass="${shoulder_mass}" radius="${shoulder_radius}" length="${shoulder_length}"/>
   </link>
   <joint name="joint_pedestal_shoulder" type="fixed">
@@ -59,15 +76,22 @@
     <visual>
       <origin xyz="${-arm_length} 0 0" rpy="${-pi / 2.0} 0 0"/>
-      <geometry><cylinder radius="${joint_radius}" length="${joint_length}"/></geometry>
+      <geometry>
+        <cylinder radius="${joint_radius}" length="${joint_length}"/>
+      </geometry>
       <material name="arm_silver"/>
     </visual>
+    <collision>
+      <origin xyz="${-arm_length} 0 0" rpy="${-pi / 2.0} 0 0"/>
+      <geometry>
+        <cylinder radius="${joint_radius}" length="${joint_length}"/>
+      </geometry>
+    </collision>
   </link>
-  <joint name="joint_shoulder_arm1" type="revolute">
+  <joint name="joint_shoulder_arm1" type="continuous">
     <parent link="shoulder_link"/>
     <child link="arm_link_1"/>
     <origin xyz="0 ${-(shoulder_length + joint_length) / 2.0} 0" rpy="0 0 0"/>
     <axis xyz="0 1 0"/>
-    <limit lower="${-joint_limit}" upper="${joint_limit}"
-           effort="${joint_effort}" velocity="${joint_velocity}"/>
+    <limit effort="${joint_effort}" velocity="${joint_velocity}"/>
     <dynamics damping="0.15" friction="0.02"/>
   </joint>
@@ -75,11 +99,10 @@
     <xacro:arm_segment length="${arm_length}" mass="0.6"/>
   </link>
-  <joint name="joint_arm1_arm2" type="revolute">
+  <joint name="joint_arm1_arm2" type="continuous">
     <parent link="arm_link_1"/>
     <child link="arm_link_2"/>
     <origin xyz="${-arm_length} ${-joint_length} 0" rpy="0 0 0"/>
     <axis xyz="0 1 0"/>
-    <limit lower="${-joint_limit}" upper="${joint_limit}"
-           effort="${joint_effort}" velocity="${joint_velocity}"/>
+    <limit effort="${joint_effort}" velocity="${joint_velocity}"/>
     <dynamics damping="0.10" friction="0.02"/>
   </joint>
@@ -88,12 +111,16 @@
     <visual>
       <origin xyz="${-end_effector_length / 2.0} 0 0" rpy="0 ${-pi / 2.0} 0"/>
-      <geometry><cylinder radius="${end_effector_radius}" length="${end_effector_length}"/></geometry>
+      <geometry>
+        <cylinder radius="${end_effector_radius}" length="${end_effector_length}"/>
+      </geometry>
       <material name="end_effector_blue"/>
     </visual>
     <collision>
       <origin xyz="${-end_effector_length / 2.0} 0 0" rpy="0 ${-pi / 2.0} 0"/>
-      <geometry><cylinder radius="${end_effector_radius}" length="${end_effector_length}"/></geometry>
+      <geometry>
+        <cylinder radius="${end_effector_radius}" length="${end_effector_length}"/>
+      </geometry>
     </collision>
-    <xacro:cylinder_inertia mass="${end_effector_mass}" radius="${end_effector_radius}" length="${end_effector_length}"/>
+    <xacro:x_aligned_cylinder_inertia origin_xyz="${-end_effector_length / 2.0} 0 0" mass="${end_effector_mass}" radius="${end_effector_radius}" length="${end_effector_length}"/>
   </link>
   <joint name="joint_arm2_end-effector" type="fixed">

File: project_6_2r_robot_arm/src/project_6_2r_robot_arm/urdf/components.xacro (robot description, xacro)
@@ -2,20 +2,20 @@
 <robot xmlns:xacro="http://www.ros.org/wiki/xacro">
   <!-- Inertia tag. -->
-  <xacro:macro name="box_inertia" params="mass x y z">
+  <xacro:macro name="box_inertia" params="origin_xyz mass base_width base_length base_height">
     <inertial>
-      <origin xyz="0 0 0" rpy="0 0 0"/>
+      <origin xyz="${origin_xyz}" rpy="0 0 0"/>
       <mass value="${mass}"/>
       <inertia
-        ixx="${mass * (y*y + z*z) / 12.0}"
+        ixx="${mass * (base_length*base_length + base_height*base_height) / 12.0}"
         ixy="0"
         ixz="0"
-        iyy="${mass * (x*x + z*z) / 12.0}"
+        iyy="${mass * (base_width*base_width + base_height*base_height) / 12.0}"
         iyz="0"
-        izz="${mass * (x*x + y*y) / 12.0}"/>
+        izz="${mass * (base_width*base_width + base_length*base_length) / 12.0}"/>
     </inertial>
   </xacro:macro>
-  <xacro:macro name="cylinder_inertia" params="mass radius length">
+  <xacro:macro name="z_aligned_cylinder_inertia" params="origin_xyz mass radius length">
     <inertial>
-      <origin xyz="0 0 0" rpy="0 0 0"/>
+      <origin xyz="${origin_xyz}" rpy="0 0 0"/>
       <mass value="${mass}"/>
       <inertia
@@ -28,14 +28,44 @@
     </inertial>
   </xacro:macro>
+  <xacro:macro name="y_aligned_cylinder_inertia" params="origin_xyz mass radius length">
+    <inertial>
+      <origin xyz="${origin_xyz}" rpy="0 0 0"/>
+      <mass value="${mass}"/>
+      <inertia
+        ixx="${mass * (3*radius*radius + length*length) / 12.0}"
+        ixy="0"
+        ixz="0"
+        iyy="${mass * radius*radius / 2.0}"
+        iyz="0"
+        izz="${mass * (3*radius*radius + length*length) / 12.0}"/>
+    </inertial>
+  </xacro:macro>
+  <xacro:macro name="x_aligned_cylinder_inertia" params="origin_xyz mass radius length">
+    <inertial>
+      <origin xyz="${origin_xyz}" rpy="0 0 0"/>
+      <mass value="${mass}"/>
+      <inertia
+        ixx="${mass * radius*radius / 2.0}"
+        ixy="0"
+        ixz="0"
+        iyy="${mass * (3*radius*radius + length*length) / 12.0}"
+        iyz="0"
+        izz="${mass * (3*radius*radius + length*length) / 12.0}"/>
+    </inertial>
+  </xacro:macro>
   <!-- Cylinder representing the body of the arm -->
   <xacro:macro name="arm_body" params="length radius material">
     <visual>
       <origin xyz="${-length / 2.0} 0 0" rpy="0 ${-pi / 2.0} 0"/>
-      <geometry><cylinder radius="${radius}" length="${length}"/></geometry>
+      <geometry>
+        <cylinder radius="${radius}" length="${length}"/>
+      </geometry>
       <material name="${material}"/>
     </visual>
     <collision>
       <origin xyz="${-length / 2.0} 0 0" rpy="0 ${-pi / 2.0} 0"/>
-      <geometry><cylinder radius="${radius}" length="${length}"/></geometry>
+      <geometry>
+        <cylinder radius="${radius}" length="${length}"/>
+      </geometry>
     </collision>
   </xacro:macro>
@@ -44,7 +74,15 @@
     <visual>
       <origin xyz="0 0 0" rpy="${-pi / 2.0} 0 0"/>
-      <geometry><cylinder radius="${radius}" length="${length}"/></geometry>
+      <geometry>
+        <cylinder radius="${radius}" length="${length}"/>
+      </geometry>
       <material name="${material}"/>
     </visual>
+    <collision>
+      <origin xyz="0 0 0" rpy="${-pi / 2.0} 0 0"/>
+      <geometry>
+        <cylinder radius="${radius}" length="${length}"/>
+      </geometry>
+    </collision>
   </xacro:macro>
   <!-- Rotating arm segment and its circular mounting flange. -->
@@ -52,5 +90,5 @@
     <xacro:arm_joint_disc radius="${joint_radius}" length="${joint_length}" material="arm_silver"/>
     <xacro:arm_body length="${length}" radius="${arm_radius}" material="arm_silver"/>
-    <xacro:cylinder_inertia mass="${mass}" radius="${arm_radius}" length="${length}"/>
+    <xacro:x_aligned_cylinder_inertia origin_xyz="${-length / 2.0} 0 0" mass="${mass}" radius="${arm_radius}" length="${length}"/>
   </xacro:macro>
 </robot>

File: project_6_2r_robot_arm/src/project_6_2r_robot_arm/urdf/properties.xacro (robot description, xacro)
@@ -11,4 +11,5 @@
   <xacro:property name="shoulder_length" value="0.15"/>
   <xacro:property name="shoulder_radius" value="0.05"/>
+  <xacro:property name="shoulder_mass" value="1.0"/>"
   <xacro:property name="arm_length" value="0.3"/>
   <xacro:property name="arm_radius" value="0.025"/>
@@ -19,5 +20,4 @@
   <xacro:property name="end_effector_radius" value="0.025"/>
   <xacro:property name="end_effector_mass" value="0.1"/>
-  <xacro:property name="joint_limit" value="${pi}"/>
   <xacro:property name="joint_effort" value="20.0"/>
   <xacro:property name="joint_velocity" value="1.5"/>

Commit message: Update robot arm positions

File: project_6_2r_robot_arm/src/project_6_2r_robot_arm/urdf/2r_robot_arm.urdf.xacro (robot description, xacro)
@@ -68,5 +68,5 @@
     <parent link="pedestal_link"/>
     <child link="shoulder_link"/>
-    <origin xyz="0 ${-shoulder_length / 4.0} ${base_height + pedestal_height}"/>
+    <origin xyz="0 ${shoulder_length / 4.0} ${base_height + pedestal_height}"/>
   </joint>
   <!-- Both rotation axes point along +Y, producing motion in the X-Z plane. -->
@@ -75,5 +75,5 @@
     <!-- Elbow housing, located at the far end of link 1. -->
     <visual>
-      <origin xyz="${-arm_length} 0 0" rpy="${-pi / 2.0} 0 0"/>
+      <origin xyz="${arm_length} 0 0" rpy="${-pi / 2.0} 0 0"/>
       <geometry>
         <cylinder radius="${joint_radius}" length="${joint_length}"/>
@@ -82,5 +82,5 @@
     </visual>
     <collision>
-      <origin xyz="${-arm_length} 0 0" rpy="${-pi / 2.0} 0 0"/>
+      <origin xyz="${arm_length} 0 0" rpy="${-pi / 2.0} 0 0"/>
       <geometry>
         <cylinder radius="${joint_radius}" length="${joint_length}"/>
@@ -91,5 +91,5 @@
     <parent link="shoulder_link"/>
     <child link="arm_link_1"/>
-    <origin xyz="0 ${-(shoulder_length + joint_length) / 2.0} 0" rpy="0 0 0"/>
+    <origin xyz="0 ${(shoulder_length + joint_length) / 2.0} 0" rpy="0 0 0"/>
     <axis xyz="0 1 0"/>
     <limit effort="${joint_effort}" velocity="${joint_velocity}"/>
@@ -102,5 +102,5 @@
     <parent link="arm_link_1"/>
     <child link="arm_link_2"/>
-    <origin xyz="${-arm_length} ${-joint_length} 0" rpy="0 0 0"/>
+    <origin xyz="${arm_length} ${joint_length} 0" rpy="0 0 0"/>
     <axis xyz="0 1 0"/>
     <limit effort="${joint_effort}" velocity="${joint_velocity}"/>
@@ -110,5 +110,5 @@
   <link name="end_effector_link">
     <visual>
-      <origin xyz="${-end_effector_length / 2.0} 0 0" rpy="0 ${-pi / 2.0} 0"/>
+      <origin xyz="${end_effector_length / 2.0} 0 0" rpy="0 ${-pi / 2.0} 0"/>
       <geometry>
         <cylinder radius="${end_effector_radius}" length="${end_effector_length}"/>
@@ -117,15 +117,15 @@
     </visual>
     <collision>
-      <origin xyz="${-end_effector_length / 2.0} 0 0" rpy="0 ${-pi / 2.0} 0"/>
+      <origin xyz="${end_effector_length / 2.0} 0 0" rpy="0 ${-pi / 2.0} 0"/>
       <geometry>
         <cylinder radius="${end_effector_radius}" length="${end_effector_length}"/>
       </geometry>
     </collision>
-    <xacro:x_aligned_cylinder_inertia origin_xyz="${-end_effector_length / 2.0} 0 0" mass="${end_effector_mass}" radius="${end_effector_radius}" length="${end_effector_length}"/>
+    <xacro:x_aligned_cylinder_inertia origin_xyz="${end_effector_length / 2.0} 0 0" mass="${end_effector_mass}" radius="${end_effector_radius}" length="${end_effector_length}"/>
   </link>
   <joint name="joint_arm2_end-effector" type="fixed">
     <parent link="arm_link_2"/>
     <child link="end_effector_link"/>
-    <origin xyz="${-arm_length} 0 0" rpy="0 0 0"/>
+    <origin xyz="${arm_length} 0 0" rpy="0 0 0"/>
   </joint>
 </robot>

File: project_6_2r_robot_arm/src/project_6_2r_robot_arm/urdf/components.xacro (robot description, xacro)
@@ -57,5 +57,5 @@
   <xacro:macro name="arm_body" params="length radius material">
     <visual>
-      <origin xyz="${-length / 2.0} 0 0" rpy="0 ${-pi / 2.0} 0"/>
+      <origin xyz="${length / 2.0} 0 0" rpy="0 ${-pi / 2.0} 0"/>
       <geometry>
         <cylinder radius="${radius}" length="${length}"/>
@@ -64,5 +64,5 @@
     </visual>
     <collision>
-      <origin xyz="${-length / 2.0} 0 0" rpy="0 ${-pi / 2.0} 0"/>
+      <origin xyz="${length / 2.0} 0 0" rpy="0 ${-pi / 2.0} 0"/>
       <geometry>
         <cylinder radius="${radius}" length="${length}"/>

Commit message: Fix small bugs

File: project_6_2r_robot_arm/src/project_6_2r_robot_arm/urdf/2r_robot_arm.urdf.xacro (robot description, xacro)
@@ -92,5 +92,5 @@
     <child link="arm_link_1"/>
     <origin xyz="0 ${(shoulder_length + joint_length) / 2.0} 0" rpy="0 0 0"/>
-    <axis xyz="0 1 0"/>
+    <axis xyz="0 -1 0"/>
     <limit effort="${joint_effort}" velocity="${joint_velocity}"/>
     <dynamics damping="0.15" friction="0.02"/>
@@ -103,5 +103,5 @@
     <child link="arm_link_2"/>
     <origin xyz="${arm_length} ${joint_length} 0" rpy="0 0 0"/>
-    <axis xyz="0 1 0"/>
+    <axis xyz="0 -1 0"/>
     <limit effort="${joint_effort}" velocity="${joint_velocity}"/>
     <dynamics damping="0.10" friction="0.02"/>

File: project_6_2r_robot_arm/src/project_6_2r_robot_arm/urdf/components.xacro (robot description, xacro)
@@ -90,5 +90,5 @@
     <xacro:arm_joint_disc radius="${joint_radius}" length="${joint_length}" material="arm_silver"/>
     <xacro:arm_body length="${length}" radius="${arm_radius}" material="arm_silver"/>
-    <xacro:x_aligned_cylinder_inertia origin_xyz="${-length / 2.0} 0 0" mass="${mass}" radius="${arm_radius}" length="${length}"/>
+    <xacro:x_aligned_cylinder_inertia origin_xyz="${length / 2.0} 0 0" mass="${mass}" radius="${arm_radius}" length="${length}"/>
   </xacro:macro>
 </robot>
