Commit message: Add an arm that rotates about the Z axis so the arm can move in 3D space

File: project_6_3r_robot_arm/src/project_6_3r_robot_arm/urdf/3r_robot_arm.urdf.xacro (robot description, xacro)
@@ -1,4 +1,4 @@
 <?xml version="1.0"?>
-<robot name="2r_robot_arm" xmlns:xacro="http://www.ros.org/wiki/xacro">
+<robot name="3r_robot_arm" xmlns:xacro="http://www.ros.org/wiki/xacro">
   <xacro:include filename="properties.xacro"/>
   <xacro:include filename="components.xacro"/>
@@ -29,5 +29,5 @@
   <link name="pedestal_link">
     <visual>
-      <origin xyz="0 0 ${base_height + pedestal_height / 2.0}"/>
+      <origin xyz="0 0 ${pedestal_height / 2.0}"/>
       <geometry>
         <cylinder length="${pedestal_height}" radius="${pedestal_radius}"/>
@@ -36,42 +36,24 @@
     </visual>
     <collision>
-      <origin xyz="0 0 ${base_height + pedestal_height / 2.0}"/>
+      <origin xyz="0 0 ${pedestal_height / 2.0}"/>
       <geometry>
         <cylinder length="${pedestal_height}" radius="${pedestal_radius}"/>
       </geometry>
     </collision>
-    <xacro:z_aligned_cylinder_inertia origin_xyz="0 0 ${base_height + pedestal_height / 2.0}" mass="${pedestal_mass}" radius="${pedestal_radius}" length="${pedestal_height}"/>
+    <xacro:z_aligned_cylinder_inertia
+      origin_xyz="0 0 ${pedestal_height / 2.0}"
+      mass="${pedestal_mass}"
+      radius="${pedestal_radius}"
+      length="${pedestal_height}"/>
   </link>
   <joint name="joint_base_pedestal" type="fixed">
     <parent link="base_link"/>
     <child link="pedestal_link"/>
-    <origin xyz="0 0 0" rpy="0 0 0"/>
+    <origin xyz="0 0 ${base_height}" rpy="0 0 0"/>
   </joint>
-  <!-- Circular shoulder pivot housing is fixed to the pedestal. -->
-  <link name="shoulder_link">
-    <visual>
-      <origin xyz="0 0 0" rpy="${pi / 2.0} 0 0"/>
-      <geometry>
-        <cylinder radius="${shoulder_radius}" length="${shoulder_length}"/>
-      </geometry>
-      <material name="joint_dark"/>
-    </visual>
-    <collision>
-      <origin xyz="0 0 0" rpy="${pi / 2.0} 0 0"/>
-      <geometry>
-        <cylinder radius="${shoulder_radius}" length="${shoulder_length}"/>
-      </geometry>
-    </collision>
-    <xacro:y_aligned_cylinder_inertia origin_xyz="0 0 0" mass="${shoulder_mass}" radius="${shoulder_radius}" length="${shoulder_length}"/>
-  </link>
-  <joint name="joint_pedestal_shoulder" type="fixed">
-    <parent link="pedestal_link"/>
-    <child link="shoulder_link"/>
-    <origin xyz="0 ${shoulder_length / 4.0} ${base_height + pedestal_height}"/>
-  </joint>
-  <!-- Both rotation axes point along +Y, producing motion in the X-Z plane. -->
+  <!-- Circular shoulder pivot housing is rotates about the Z axis. -->
   <link name="arm_link_1">
-    <xacro:arm_segment length="${arm_length}" mass="${arm_mass}"/>
-    <!-- Elbow housing, located at the far end of link 1. -->
+    <xacro:arm_segment length="${arm_length}" mass="${arm_mass}" joint_axis="z"/>
+    <!-- Shoulder housing, located at the far end of link 1. -->
     <visual>
       <origin xyz="${arm_length} 0 0" rpy="${-pi / 2.0} 0 0"/>
@@ -88,14 +70,29 @@
     </collision>
   </link>
-  <joint name="joint_shoulder_arm1" type="continuous">
-    <parent link="shoulder_link"/>
+  <joint name="joint_pedestal_arm1" type="continuous">
+    <parent link="pedestal_link"/>
     <child link="arm_link_1"/>
-    <origin xyz="0 ${(shoulder_length + joint_length) / 2.0} 0" rpy="0 0 0"/>
-    <axis xyz="0 -1 0"/>
+    <origin xyz="0 0 ${pedestal_height}" rpy="0 0 0"/>
+    <axis xyz="0 0 1"/>
     <limit effort="${joint_effort}" velocity="${joint_velocity}"/>
     <dynamics damping="0.15" friction="0.02"/>
   </joint>
+  <!-- Planar arm. Both joints rotate about the same axis -->
   <link name="arm_link_2">
-    <xacro:arm_segment length="${arm_length}" mass="0.6"/>
+    <xacro:arm_segment length="${arm_length}" mass="${arm_mass}"/>
+    <!-- Elbow housing, located at the far end of link 2. -->
+    <visual>
+      <origin xyz="${arm_length} 0 0" rpy="${-pi / 2.0} 0 0"/>
+      <geometry>
+        <cylinder radius="${joint_radius}" length="${joint_length}"/>
+      </geometry>
+      <material name="arm_silver"/>
+    </visual>
+    <collision>
+      <origin xyz="${arm_length} 0 0" rpy="${-pi / 2.0} 0 0"/>
+      <geometry>
+        <cylinder radius="${joint_radius}" length="${joint_length}"/>
+      </geometry>
+    </collision>
   </link>
   <joint name="joint_arm1_arm2" type="continuous">
@@ -103,5 +100,16 @@
     <child link="arm_link_2"/>
     <origin xyz="${arm_length} ${joint_length} 0" rpy="0 0 0"/>
-    <axis xyz="0 -1 0"/>
+    <axis xyz="0 1 0"/>
+    <limit effort="${joint_effort}" velocity="${joint_velocity}"/>
+    <dynamics damping="0.15" friction="0.02"/>
+  </joint>
+  <link name="arm_link_3">
+    <xacro:arm_segment length="${arm_length}" mass="0.6"/>
+  </link>
+  <joint name="joint_arm2_arm3" type="continuous">
+    <parent link="arm_link_2"/>
+    <child link="arm_link_3"/>
+    <origin xyz="${arm_length} ${joint_length} 0" rpy="0 0 0"/>
+    <axis xyz="0 1 0"/>
     <limit effort="${joint_effort}" velocity="${joint_velocity}"/>
     <dynamics damping="0.10" friction="0.02"/>
@@ -125,5 +133,5 @@
   </link>
   <joint name="joint_arm2_end-effector" type="fixed">
-    <parent link="arm_link_2"/>
+    <parent link="arm_link_3"/>
     <child link="end_effector_link"/>
     <origin xyz="${arm_length} 0 0" rpy="0 0 0"/>

File: project_6_3r_robot_arm/src/project_6_3r_robot_arm/urdf/components.xacro (robot description, xacro)
@@ -87,6 +87,23 @@
   </xacro:macro>
   <!-- Rotating arm segment and its circular mounting flange. -->
-  <xacro:macro name="arm_segment" params="length mass">
-    <xacro:arm_joint_disc radius="${joint_radius}" length="${joint_length}" material="arm_silver"/>
+  <xacro:macro name="arm_segment" params="length mass joint_axis:='y'">
+    <xacro:if value="${joint_axis == 'z'}">
+      <visual>
+        <origin xyz="0 0 0" rpy="0 0 0"/>
+        <geometry>
+          <cylinder radius="${joint_radius}" length="${joint_length}"/>
+        </geometry>
+        <material name="arm_silver"/>
+      </visual>
+      <collision>
+        <origin xyz="0 0 0" rpy="0 0 0"/>
+        <geometry>
+          <cylinder radius="${joint_radius}" length="${joint_length}"/>
+        </geometry>
+      </collision>
+    </xacro:if>
+    <xacro:unless value="${joint_axis == 'z'}">
+      <xacro:arm_joint_disc radius="${joint_radius}" length="${joint_length}" material="arm_silver"/>
+    </xacro:unless>
     <xacro:arm_body length="${length}" radius="${arm_radius}" material="arm_silver"/>
     <xacro:x_aligned_cylinder_inertia origin_xyz="${length / 2.0} 0 0" mass="${mass}" radius="${arm_radius}" length="${length}"/>

File: project_6_3r_robot_arm/src/project_6_3r_robot_arm/urdf/properties.xacro (robot description, xacro)
@@ -9,12 +9,9 @@
   <xacro:property name="pedestal_radius" value="0.035"/>
   <xacro:property name="pedestal_mass" value="2.0"/>
-  <xacro:property name="shoulder_length" value="0.15"/>
-  <xacro:property name="shoulder_radius" value="0.05"/>
-  <xacro:property name="shoulder_mass" value="1.0"/>"
   <xacro:property name="arm_length" value="0.3"/>
-  <xacro:property name="arm_radius" value="0.025"/>
+  <xacro:property name="arm_radius" value="0.035"/>
   <xacro:property name="arm_mass" value="0.8"/>
-  <xacro:property name="joint_radius" value="0.05"/>
-  <xacro:property name="joint_length" value="0.05"/>
+  <xacro:property name="joint_radius" value="0.04"/>
+  <xacro:property name="joint_length" value="0.085"/>
   <xacro:property name="end_effector_length" value="0.05"/>
   <xacro:property name="end_effector_radius" value="0.025"/>
@@ -23,5 +20,4 @@
   <xacro:property name="joint_velocity" value="1.5"/>
   <material name="base_gray"><color rgba="0.25 0.29 0.33 1"/></material>
-  <material name="joint_dark"><color rgba="0.12 0.14 0.18 1"/></material>
   <material name="arm_silver"><color rgba="0.72 0.77 0.81 1"/></material>
   <material name="end_effector_blue"><color rgba="0 0 1 1"/></material>
